File: touch_button_tester/touch_button_tester.sch (KiCad schematic (older format))
At the start: 21 parts

Commit message: updated schematic
Parts:
- gave numbers to parts that had none: 21

Commit message: finished pcb; gerber files creaeted
Parts:
- C1, C2, C3, C4, C5, C6: footprint (none) -> Capacitor_SMD:C_0805_2012Metric_Pad1.15x1.40mm_HandSolder
- D1, D2, D3, D4: footprint (none) -> LED_SMD:LED_0805_2012Metric_Castellated
- J1: footprint (none) -> Connector_PinHeader_2.54mm:PinHeader_1x05_P2.54mm_Vertical
- R1, R2, R3, R4: footprint (none) -> Resistor_SMD:R_0805_2012Metric_Pad1.15x1.40mm_HandSolder
- U1, U2, U3: footprint (none) -> touch_button:touch_button
- U4, U5, U6: footprint MODULE -> Package_TO_SOT_SMD:SOT-23-6_Handsoldering
Changed lines of the file:
@@
 F 0 "U4" H 5200 1715 50  0000 C CNN
 F 1 "ttp223" H 5200 1624 50  0000 C CNN
-F 2 "MODULE" H 5200 1250 50  0001 C CNN
+F 2 "Package_TO_SOT_SMD:SOT-23-6_Handsoldering" H 5200 1250 50  0001 C CNN
 F 3 "DOCUMENTATION" H 5200 1250 50  0001 C CNN
 	1    5200 1250
@@
 F 0 "U1" H 3908 1665 50  0000 C CNN
 F 1 "touch_button" H 3908 1574 50  0000 C CNN
-F 2 "" H 3850 1350 50  0001 C CNN
+F 2 "touch_button:touch_button" H 3850 1350 50  0001 C CNN
 F 3 "" H 3850 1350 50  0001 C CNN
 	1    3850 1350
@@
 F 0 "J1" H 1300 2450 50  0000 C CNN
 F 1 "I/O" H 1300 2350 50  0000 C CNN
-F 2 "" H 1200 2000 50  0001 C CNN
+F 2 "Connector_PinHeader_2.54mm:PinHeader_1x05_P2.54mm_Vertical" H 1200 2000 50  0001 C CNN
 F 3 "~" H 1200 2000 50  0001 C CNN
 	1    1200 2000
@@
 F 0 "D1" V 1296 2880 50  0000 R CNN
 F 1 "t1" V 1205 2880 50  0000 R CNN
-F 2 "" V 1250 2950 50  0001 C CNN
+F 2 "LED_SMD:LED_0805_2012Metric_Castellated" V 1250 2950 50  0001 C CNN
 F 3 "~" V 1250 2950 50  0001 C CNN
 	1    1250 2950
@@
 F 0 "D2" V 1546 2880 50  0000 R CNN
 F 1 "t2" V 1455 2880 50  0000 R CNN
-F 2 "" V 1500 2950 50  0001 C CNN
+F 2 "LED_SMD:LED_0805_2012Metric_Castellated" V 1500 2950 50  0001 C CNN
 F 3 "~" V 1500 2950 50  0001 C CNN
 	1    1500 2950
@@
 F 0 "D3" V 1796 2880 50  0000 R CNN
 F 1 "t3" V 1705 2880 50  0000 R CNN
-F 2 "" V 1750 2950 50  0001 C CNN
+F 2 "LED_SMD:LED_0805_2012Metric_Castellated" V 1750 2950 50  0001 C CNN
 F 3 "~" V 1750 2950 50  0001 C CNN
 	1    1750 2950
@@
 F 0 "D4" V 2046 2880 50  0000 R CNN
 F 1 "pwr" V 1955 2880 50  0000 R CNN
-F 2 "" V 2000 2950 50  0001 C CNN
+F 2 "LED_SMD:LED_0805_2012Metric_Castellated" V 2000 2950 50  0001 C CNN
 F 3 "~" V 2000 2950 50  0001 C CNN
 	1    2000 2950
@@
 F 0 "R1" H 1309 3296 50  0000 L CNN
 F 1 "2k2" H 1309 3205 50  0000 L CNN
-F 2 "" H 1250 3250 50  0001 C CNN
+F 2 "Resistor_SMD:R_0805_2012Metric_Pad1.15x1.40mm_HandSolder" H 1250 3250 50  0001 C CNN
 F 3 "~" H 1250 3250 50  0001 C CNN
 	1    1250 3250
@@
 F 0 "R2" H 1559 3296 50  0000 L CNN
 F 1 "2k2" H 1559 3205 50  0000 L CNN
-F 2 "" H 1500 3250 50  0001 C CNN
+F 2 "Resistor_SMD:R_0805_2012Metric_Pad1.15x1.40mm_HandSolder" H 1500 3250 50  0001 C CNN
 F 3 "~" H 1500 3250 50  0001 C CNN
 	1    1500 3250
@@
 F 0 "R3" H 1809 3296 50  0000 L CNN
 F 1 "2k2" H 1809 3205 50  0000 L CNN
-F 2 "" H 1750 3250 50  0001 C CNN
+F 2 "Resistor_SMD:R_0805_2012Metric_Pad1.15x1.40mm_HandSolder" H 1750 3250 50  0001 C CNN
 F 3 "~" H 1750 3250 50  0001 C CNN
 	1    1750 3250
@@
 F 0 "R4" H 2059 3296 50  0000 L CNN
 F 1 "2k2" H 2059 3205 50  0000 L CNN
-F 2 "" H 2000 3250 50  0001 C CNN
+F 2 "Resistor_SMD:R_0805_2012Metric_Pad1.15x1.40mm_HandSolder" H 2000 3250 50  0001 C CNN
 F 3 "~" H 2000 3250 50  0001 C CNN
 	1    2000 3250
@@
 F 0 "C4" H 5992 1446 50  0000 L CNN
 F 1 "100n" H 5992 1355 50  0000 L CNN
-F 2 "" H 5900 1400 50  0001 C CNN
+F 2 "Capacitor_SMD:C_0805_2012Metric_Pad1.15x1.40mm_HandSolder" H 5900 1400 50  0001 C CNN
 F 3 "~" H 5900 1400 50  0001 C CNN
 	1    5900 1400
@@
 F 0 "C1" H 4342 1596 50  0000 L CNN
 F 1 "0..50p" H 4342 1505 50  0000 L CNN
-F 2 "" H 4250 1550 50  0001 C CNN
+F 2 "Capacitor_SMD:C_0805_2012Metric_Pad1.15x1.40mm_HandSolder" H 4250 1550 50  0001 C CNN
 F 3 "~" H 4250 1550 50  0001 C CNN
 	1    4250 1550
@@
 F 0 "U5" H 5200 2915 50  0000 C CNN
 F 1 "ttp223" H 5200 2824 50  0000 C CNN
-F 2 "MODULE" H 5200 2450 50  0001 C CNN
+F 2 "Package_TO_SOT_SMD:SOT-23-6_Handsoldering" H 5200 2450 50  0001 C CNN
 F 3 "DOCUMENTATION" H 5200 2450 50  0001 C CNN
 	1    5200 2450
@@
 F 0 "U2" H 3908 2865 50  0000 C CNN
 F 1 "touch_button" H 3908 2774 50  0000 C CNN
-F 2 "" H 3850 2550 50  0001 C CNN
+F 2 "touch_button:touch_button" H 3850 2550 50  0001 C CNN
 F 3 "" H 3850 2550 50  0001 C CNN
 	1    3850 2550
@@
 F 0 "C5" H 5992 2646 50  0000 L CNN
 F 1 "100n" H 5992 2555 50  0000 L CNN
-F 2 "" H 5900 2600 50  0001 C CNN
+F 2 "Capacitor_SMD:C_0805_2012Metric_Pad1.15x1.40mm_HandSolder" H 5900 2600 50  0001 C CNN
 F 3 "~" H 5900 2600 50  0001 C CNN
 	1    5900 2600
@@
 F 0 "C2" H 4342 2796 50  0000 L CNN
 F 1 "0..50p" H 4342 2705 50  0000 L CNN
-F 2 "" H 4250 2750 50  0001 C CNN
+F 2 "Capacitor_SMD:C_0805_2012Metric_Pad1.15x1.40mm_HandSolder" H 4250 2750 50  0001 C CNN
 F 3 "~" H 4250 2750 50  0001 C CNN
 	1    4250 2750
@@
 F 0 "U6" H 5200 4115 50  0000 C CNN
 F 1 "ttp223" H 5200 4024 50  0000 C CNN
-F 2 "MODULE" H 5200 3650 50  0001 C CNN
+F 2 "Package_TO_SOT_SMD:SOT-23-6_Handsoldering" H 5200 3650 50  0001 C CNN
 F 3 "DOCUMENTATION" H 5200 3650 50  0001 C CNN
 	1    5200 3650
@@
 F 0 "U3" H 3908 4065 50  0000 C CNN
 F 1 "touch_button" H 3908 3974 50  0000 C CNN
-F 2 "" H 3850 3750 50  0001 C CNN
+F 2 "touch_button:touch_button" H 3850 3750 50  0001 C CNN
 F 3 "" H 3850 3750 50  0001 C CNN
 	1    3850 3750
@@
 F 0 "C6" H 5992 3846 50  0000 L CNN
 F 1 "100n" H 5992 3755 50  0000 L CNN
-F 2 "" H 5900 3800 50  0001 C CNN
+F 2 "Capacitor_SMD:C_0805_2012Metric_Pad1.15x1.40mm_HandSolder" H 5900 3800 50  0001 C CNN
 F 3 "~" H 5900 3800 50  0001 C CNN
 	1    5900 3800
@@
 F 0 "C3" H 4342 3996 50  0000 L CNN
 F 1 "0..50p" H 4342 3905 50  0000 L CNN
-F 2 "" H 4250 3950 50  0001 C CNN
+F 2 "Capacitor_SMD:C_0805_2012Metric_Pad1.15x1.40mm_HandSolder" H 4250 3950 50  0001 C CNN
 F 3 "~" H 4250 3950 50  0001 C CNN
 	1    4250 3950
